File: 99_Resources/KiCad/03_SonarRangeDetector/03_SonarRangeDetector.kicad_sch (KiCad schematic)
At the start: 12 parts

Commit message: don't point at KiCad V5 libraries
Parts:
- removed A?: Arduino_USB, symbol mdoLibrary:Arduino_USB
- removed M?: HC-SR04, symbol mdoLibrary:HC-SR04
- added A1: Arduino_USB, symbol MDO:Arduino_USB
- added M1: HC-SR04, symbol MDO:HC-SR04
Connections:
- net at R?.2: now also A1.~ (VIN)
- net at SW?.1: now also A1.~ (VIN)
- net at SW?.2: now also A1.~ (VIN), M1.~ (VCC)
- net at D?.1 (VDD), D?.1 (VDD), D?.1 (VDD)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: now also A1.~ (VIN), M1.~ (VCC)
- net at D?.3 (VSS), D?.3 (VSS), D?.3 (VSS)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: now also A1.~ (VIN)
- new net: A1.~ (VIN), M1.~ (VCC) (x2)
Changed lines of the file:
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@@
-    )
-  )
-  (symbol (lib_id "mdoLibrary:Arduino_USB") (at 137.16 130.81 0) (unit 1)
-    (in_bom yes) (on_board yes) (dnp no)
-    (property "Reference" "A?" (at 137.16 105.7402 0)
-      (effects (font (size 1.524 1.524)))
-    )
-    (property "Value" "Arduino_USB" (at 137.16 108.4326 0)
-      (effects (font (size 1.524 1.524)))
-    )
-    (property "Footprint" "" (at 137.16 130.81 0)
-      (effects (font (size 1.524 1.524)))
-    )
-    (property "Datasheet" "" (at 137.16 130.81 0)
-      (effects (font (size 1.524 1.524)))
-    )
-    (instances
-      (project "03_SonarRangeDetector"
-        (path "/5d688ce1-536d-4657-be00-f47641c4df42"
-          (reference "A?") (unit 1)
-        )
-      )
     )
   )
@@
     )
   )
-  (symbol (lib_id "mdoLibrary:HC-SR04") (at 80.01 140.97 0) (unit 1)
-    (in_bom yes) (on_board yes) (dnp no)
-    (property "Reference" "M?" (at 84.0232 138.049 0)
+  (symbol (lib_id "MDO:HC-SR04") (at 80.01 140.97 0) (unit 1)
+    (in_bom yes) (on_board yes) (dnp no) (fields_autoplaced)
+    (property "Reference" "M1" (at 81.915 138.43 0)
       (effects (font (size 1.27 1.27)))
     )
-    (property "Value" "HC-SR04" (at 84.0232 140.3604 0)
+    (property "Value" "HC-SR04" (at 81.915 140.97 0)
       (effects (font (size 1.27 1.27)))
     )
@@
       (effects (font (size 1.27 1.27)) hide)
     )
-    (instances
-      (project "03_SonarRangeDetector"
-        (path "/5d688ce1-536d-4657-be00-f47641c4df42"
-          (reference "M?") (unit 1)
-        )
-      )
+    (pin "~")
+    (pin "~")
+    (pin "~")
+    (pin "~")
+    (instances
+      (project "03_SonarRangeDetector"
+        (path "/5d688ce1-536d-4657-be00-f47641c4df42"
+          (reference "M1") (unit 1)
+        )
+      )
+    )
+  )
+  (symbol (lib_id "MDO:Arduino_USB") (at 137.16 130.81 0) (unit 1)
+    (in_bom yes) (on_board yes) (dnp no) (fields_autoplaced)
+    (property "Reference" "A1" (at 136.525 106.68 0)
+      (effects (font (size 1.524 1.524)))
+    )
+    (property "Value" "Arduino_USB" (at 136.525 109.22 0)
+      (effects (font (size 1.524 1.524)))
+    )
+    (property "Footprint" "" (at 137.16 130.81 0)
+      (effects (font (size 1.524 1.524)))
+    )
+    (property "Datasheet" "" (at 137.16 130.81 0)
+      (effects (font (size 1.524 1.524)))
+    )
+    (pin "~")
+    (pin "~")
+    (pin "~")
+    (pin "~")
+    (pin "~")
+    (pin "~")
+    (pin "~")
+    (pin "~")
+    (pin "~")
+    (pin "~")
+    (pin "~")
+    (pin "~")
+    (pin "~")
+    (pin "~")
+    (pin "~")
+    (pin "~")
+    (pin "~")
+    (pin "~")
+    (pin "~")
+    (pin "~")
+    (pin "~")
+    (pin "~")
+    (pin "~")
+    (pin "~")
+    (pin "~")
+    (pin "~")
+    (pin "~")
+    (pin "~")
+    (pin "~")
+    (pin "~")
+    (instances
+      (project "03_SonarRangeDetector"
+        (path "/5d688ce1-536d-4657-be00-f47641c4df42"
+          (reference "A1") (unit 1)
+        )
+      )
