File: 99_Resources/KiCad/04_DemoReelSound/04_DemoReelSound.kicad_sch (KiCad schematic)
At the start: 11 parts, among them J1 Conn_01x03_Pin, J4 Conn_01x03_Socket, U1 BlueToothAudioR

Commit message: minor tweaks
Connections:
- net at A?.~ (VIN): now also A1.~ (USB-_15)
- net at A1.~ (USB-_15): no longer A?.~ (VIN)
- net at Z?.~ (GND): now also A1.~ (USB-_15), U1.~ (TX)
- net at U1.~ (TX): now also J4.2 (Pin_2)
- new net: A?.~ (VIN), M?.~ (VCC), SW?.2
- new net: A?.~ (VIN), M?.~ (VCC) (x2)
- new net: A1.~ (USB-_15), A?.~ (VIN), J4.3 (Pin_3), U1.~ (TX), Z?.~ (GND)
- new net: A1.~ (USB-_15), A?.~ (VIN)
- new net: A1.~ (USB-_15), U1.~ (TX) (x3)
- now unconnected: A1.~ (USB-_15), A1.~ (USB-_15), A1.~ (USB-_15), A1.~ (USB-_15), A1.~ (USB-_15), A1.~ (USB-_15)
