File: 99_Resources/KiCad/04_DemoReelVoiceCommand_UART/04_DemoReelVoiceCommand.kicad_sch (KiCad schematic)
At the start: 11 parts, among them J1 Conn_01x03_Pin, J4 Conn_01x03_Socket, M1 SEN0539_VoiceCommand, U1 BlueToothAudioR

Commit message: more I2C
Connections:
- net at A?.~ (VIN): now also A3.~ (VIN)
- net at A1.~ (USB-_15): no longer A?.~ (VIN)
- net at A3.~ (VIN): no longer A?.~ (VIN)
- net at Z?.~ (GND): now also A1.~ (USB-_15), A3.~ (VIN), M1.~ (VCC_RED), U1.~ (TX)
- net at U1.~ (TX): now also J4.2 (Pin_2)
- new net: A1.~ (USB-_15), A3.~ (VIN), A?.~ (VIN), J4.3 (Pin_3), M1.~ (VCC_RED), U1.~ (TX), Z?.~ (GND)
- new net: A1.~ (USB-_15), A?.~ (VIN) (x2)
- new net: A3.~ (VIN), A?.~ (VIN) (x3)
- new net: A1.~ (USB-_15), U1.~ (TX) (x3)
- new net: A3.~ (VIN), M1.~ (VCC_RED)
- now unconnected: A1.~ (USB-_15), A1.~ (USB-_15), A1.~ (USB-_15), A1.~ (USB-_15), A1.~ (USB-_15), A1.~ (USB-_15), A3.~ (VIN), A3.~ (VIN), A3.~ (VIN), A3.~ (VIN), A3.~ (VIN), A3.~ (VIN)
Changed lines of the file:
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@@
-    (stroke (width 0) (type default))
-  )
-  (wire (pts (xy 151.13 96.52) (xy 151.13 139.7))
     (stroke (width 0) (type default))
   )
@@
     (stroke (width 0) (type default))
   )
-  (wire (pts (xy 146.05 96.52) (xy 151.13 96.52))
-    (stroke (width 0) (type default))
-  )
