File: 99_Resources/KiCad/04_DemoReelVoiceCommand_UART/ProgramingArduino.kicad_sch (KiCad schematic)
At the start: 1 part

Commit message: updates to UART and I2C versions of KiCad DemoReelVoiceCommand
Other:
- company: (none) -> Author: https://github.com/Mark-MDO47/ArduinoClass
- title: ProgrammingArduino -> 04 The Finale - DemoReelVoiceCommand_UART
Changed lines of the file:
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@@
   (paper "USLetter")
   (title_block
-    (title "ProgrammingArduino")
-    (date "2023-07-23")
+    (title "04 The Finale - DemoReelVoiceCommand_UART")
+    (date "2023-08-06")
+    (company "Author: https://github.com/Mark-MDO47/ArduinoClass")
     (comment 1 "for code: https://github.com/Mark-MDO47/BluetoothAudioTransmitter_KCX_BT_EMITTER")
   )
