File: 99_Resources/KiCad/99_ChristmasTree/99_ChristmasTree.kicad_sch (KiCad schematic)
At the start: 9 parts, among them M1 SEN0539_VoiceCommand

Commit message: KiCad - make it neater
Parts:
- added SW1: SW_SPST, symbol MDO:SW_SPST
Connections:
- net at A?.~ (VIN): now also A3.~ (VIN)
- net at A3.~ (VIN): no longer A?.~ (VIN)
- net at BT?.1 (+): now also SW1.~ (B)
- net at Z4.~ (GND): now also Z3.~ (GND); no longer Z1.~ (GND)
- net at Z3.~ (GND): now also Z2.~ (GND); no longer Z4.~ (GND)
- new net: A3.~ (VIN), A?.~ (VIN), M1.~ (VCC_RED), Z1.~ (GND), Z2.~ (GND), Z3.~ (GND), Z4.~ (GND) (x2)
- new net: A3.~ (VIN), A?.~ (VIN) (x3)
- new net: Z1.~ (GND), Z4.~ (GND)
- new net: A3.~ (VIN), M1.~ (VCC_RED)
- now unconnected: A3.~ (VIN), A3.~ (VIN), A3.~ (VIN), A3.~ (VIN), A3.~ (VIN), A3.~ (VIN), Z1.~ (GND), Z1.~ (GND)
Other:
- moved on the sheet: BT?, R?, Z2

Commit message: use special I2C pins for Christmas Tree
Connections:
- net at A?.~ (VIN): now also A3.~ (VIN)
- net at A3.~ (VIN): no longer A?.~ (VIN)
- net at Z4.~ (GND): now also Z3.~ (GND); no longer Z1.~ (GND)
- net at Z3.~ (GND): now also Z2.~ (GND); no longer Z4.~ (GND)
- new net: A3.~ (VIN), A?.~ (VIN), M1.~ (VCC_RED), Z1.~ (GND), Z2.~ (GND), Z3.~ (GND), Z4.~ (GND) (x2)
- new net: A3.~ (VIN), A?.~ (VIN) (x3)
- new net: Z1.~ (GND), Z4.~ (GND)
- new net: A3.~ (VIN), M1.~ (VCC_RED)
- now unconnected: A3.~ (VIN), A3.~ (VIN), A3.~ (VIN), A3.~ (VIN), A3.~ (VIN), A3.~ (VIN), Z1.~ (GND), Z1.~ (GND)
Other:
- note added: "A5 & A4 are special I2C pins"
Changed lines of the file:
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@@
   (title_block
     (title "99 Christmas Tree")
-    (date "2023-12-09")
+    (date "2023-12-11")
     (company "Author: https://github.com/Mark-MDO47/ArduinoClass")
     (comment 1 "NOTE: Chips & Modules shown top view, notch at top")
@@
     (stroke (width 0) (type default))
   )
-  (wire (pts (xy 186.69 139.7) (xy 205.74 139.7))
+  (wire (pts (xy 186.69 139.7) (xy 196.85 139.7))
     (stroke (width 0) (type default))
   )
@@
     (stroke (width 0) (type default))
   )
+  (wire (pts (xy 193.04 152.4) (xy 193.04 137.16))
+    (stroke (width 0) (type default))
+  )
   (wire (pts (xy 16.51 111.76) (xy 16.51 110.49))
     (stroke (width 0) (type default))
@@
     (stroke (width 0) (type default))
   )
+  (wire (pts (xy 245.11 149.86) (xy 196.85 149.86))
+    (stroke (width 0) (type default))
+  )
   (wire (pts (xy 67.31 80.01) (xy 67.31 111.76))
     (stroke (width 0) (type default))
@@
     (stroke (width 0) (type default))
   )
-  (wire (pts (xy 198.12 137.16) (xy 198.12 134.62))
-    (stroke (width 0) (type default))
-  )
   (wire (pts (xy 110.49 119.38) (xy 205.74 119.38))
     (stroke (width 0) (type default))
@@
     (stroke (width 0) (type default))
   )
+  (wire (pts (xy 193.04 137.16) (xy 186.69 137.16))
+    (stroke (width 0) (type default))
+  )
   (wire (pts (xy 113.03 153.67) (xy 119.38 153.67))
     (stroke (width 0) (type default))
   )
+  (wire (pts (xy 236.22 121.92) (xy 245.11 121.92))
+    (stroke (width 0) (type default))
+  )
   (wire (pts (xy 67.31 80.01) (xy 114.3 80.01))
     (stroke (width 0) (type default))
   )
+  (wire (pts (xy 250.19 119.38) (xy 250.19 152.4))
+    (stroke (width 0) (type default))
+  )
   (wire (pts (xy 168.91 74.93) (xy 168.91 62.23))
     (stroke (width 0) (type default))
@@
     (stroke (width 0) (type default))
   )
-  (wire (pts (xy 198.12 134.62) (xy 205.74 134.62))
+  (wire (pts (xy 196.85 149.86) (xy 196.85 139.7))
     (stroke (width 0) (type default))
   )
@@
     (stroke (width 0) (type default))
   )
+  (wire (pts (xy 236.22 119.38) (xy 250.19 119.38))
+    (stroke (width 0) (type default))
+  )
+  (wire (pts (xy 250.19 152.4) (xy 193.04 152.4))
+    (stroke (width 0) (type default))
+  )
   (wire (pts (xy 166.37 82.55) (xy 227.33 82.55))
     (stroke (width 0) (type default))
@@
     (stroke (width 0) (type default))
   )
-  (wire (pts (xy 198.12 137.16) (xy 186.69 137.16))
-    (stroke (width 0) (type default))
-  )
   (wire (pts (xy 16.51 101.6) (xy 21.59 101.6))
+    (stroke (width 0) (type default))
+  )
+  (wire (pts (xy 245.11 121.92) (xy 245.11 149.86))
     (stroke (width 0) (type default))
   )
@@
     (effects (font (size 1.27 1.27)) (justify left bottom))
   )
+  (text "A5 & A4 are special I2C pins" (at 238.76 116.84 0)
+    (effects (font (size 1.27 1.27)) (justify left bottom))
+  )
